File: System design/V 0.1/EDA/BMS.kicad_sch (KiCad schematic)
At the start: 20 parts, among them J1 Conn_01x03_Pin, J2 Conn_01x02_Pin, Q1 NMOS, Q2 NMOS, Q3 PMOS, Q4 PMOS, U1 SN74LVC2G14DBV, U2 SN74LVC2G14DBV, U3 CDSOT236-0504C

Commit message: BMS Design Update
Connections:
- net at Q2.2 (G): now also Q1.2 (G)
Changed lines of the file:
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@@
+	(wire
+		(pts
+			(xy 118.11 58.42) (xy 118.11 72.39)
+		)
+		(stroke
+			(width 0)
+			(type default)
+		)
+	)
 	(wire
 		(pts
