File: System design/V 0.1/EDA/BMS.kicad_pcb (KiCad board)
At the start: 2 copper layers, 27.5 x 61.5 mm, 22 parts, among them J1 Conn_01x03_Pin, J2 Conn_01x02_Pin, Q1 NMOS, Q2 NMOS, Q3 PMOS, Q4 PMOS, U1 SN74LVC2G14DBV, U2 SN74LVC2G14DBV, U3 CDSOT236-0504C

Commit message: Updated BMS Design
Parts:
- moved ARTS Lab 5.84 mm to (146.3, 78.7)
- moved USC 4.61 mm to (146.5, 90.3)
Other:
- outline, holes or cut-outs redrawn
- board text added: "BM"
- board text added: "BMS 2S Module V 0.1 M. Usman Khan Md Asif Khan Date: 10/21/2025"
- board text added: "R1"
- board text removed: "Bm"
Changed lines of the file:
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@@
 		(tags "capacitor handsolder")
 		(property "Reference" "C1"
-			(at 0 -2.155 0)
+			(at -0.1947 -1.4736 0)
 			(layer "F.SilkS")
 			(effects
@@
 		(tags "connector JST EH vertical")
 		(property "Reference" "J2"
-			(at 2.6 3.75 0)
+			(at 1.5524 3.9996 0)
 			(layer "F.SilkS")
 			(effects
@@
 	(footprint "LOGO"
 		(layer "B.Cu")
-		(at 144.471682 73.140328)
+		(at 146.304 78.6892)
 		(property "Reference" "ARTS Lab"
 			(at 0 5 0)
@@
 	(footprint "LOGO"
 		(layer "B.Cu")
-		(at 144.471682 86.140328 180)
+		(at 146.5072 90.2716 180)
 		(property "Reference" "USC"
 			(at 0 -6.5 0)
@@
 	)
 	(gr_circle
-		(center 135.9916 63.431728)
-		(end 135.1704 61.932128)
+		(center 135.9916 63.634928)
+		(end 135.1704 62.135328)
 		(stroke
 			(width 0.05)
@@
 	)
 	(gr_text "B-"
-		(at 144.45 118.4 0)
+		(at 144.272 118.4656 0)
 		(layer "F.SilkS")
 		(effects
@@
 		)
 	)
+	(gr_text "R1"
+		(at 139.0396 75.5904 0)
+		(layer "F.SilkS")
+		(effects
+			(font
+				(size 1 1)
+				(thickness 0.15)
+			)
+		)
+	)
 	(gr_text "P+"
 		(at 153.65 66.55 0)
@@
 		)
 	)
-	(gr_text "Bm"
+	(gr_text "BM"
 		(at 141.15 118.4 0)
 		(layer "F.SilkS")
@@
 	)
 	(gr_text "B+"
-		(at 137.4 118.45 0)
+		(at 138.2776 118.3132 0)
 		(layer "F.SilkS")
 		(effects
@@
 		)
 	)
+	(gr_text "BMS 2S Module V 0.1\nM. Usman Khan\nMd Asif Khan\nDate: 10/21/2025"
+		(at 147.1168 105.0036 0)
+		(layer "B.SilkS")
+		(effects
+			(font
+				(size 1 1)
+				(thickness 0.1)
+			)
+			(justify bottom mirror)
+		)
+	)

Commit message: BMS Design Updated
Routing:
- net GND: vias 0 -> 32
