File: System design/V.02/EDA/_autosave-EDA.kicad_pcb (KiCad board)
At the start: 2 copper layers, 27.5 x 61.5 mm, 22 parts, among them J1 Conn_01x03_Pin, J2 Conn_01x02_Pin, Q1 NMOS, Q2 NMOS, Q3 PMOS, Q4 PMOS, U1 SN74LVC2G14DBV, U2 SN74LVC2G14DBV, U3 CDSOT236-0504C

Commit message: Update pads
Parts:
- moved C1 0.07 mm to (139.4, 73.1)
Routing:
- net Net-(J1-Pin_3): track 100.9 -> 0.00 mm
- net Net-(J1-Pin_1): track 55.1 -> 0.00 mm, vias 1 -> 0
- net Net-(Q2-D): track 42.8 -> 0.00 mm
- net Net-(J1-Pin_2): track 42.2 -> 0.00 mm
- net Net-(Q1-D): track 27.4 -> 0.00 mm, vias 2 -> 0
- net Net-(U3-VP): track 15.4 -> 0.00 mm
- net Net-(U2-GND): track 10.5 -> 0.00 mm
- net Net-(U1-GND): track 10.4 -> 0.00 mm
- net Net-(U3-IO3): track 9.63 -> 0.00 mm
- net Net-(Q1-G): track 9.58 -> 0.00 mm
- net Net-(U3-IO2): track 8.51 -> 0.00 mm
- net Net-(Q3-D): track 3.88 -> 0.00 mm
- net Net-(Q4-D): track 3.75 -> 0.00 mm
- net Net-(Q4-S): track 3.15 -> 0.00 mm
- net Net-(Q3-S): track 3.15 -> 0.00 mm
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- removed copper zone on B.Cu, net GND
- removed copper zone on F.Cu, net GND
